Commit message: add all changes

File: ABBRobots/IRB120/irb120_ros2_gazebo/urdf/irb120.urdf.xacro (robot description, xacro)
@@ -1,53 +1,4 @@
 <?xml version="1.0" ?>
-<!--
-# ===================================== COPYRIGHT ===================================== #
-#                                                                                       #
-#  IFRA (Intelligent Flexible Robotics and Assembly) Group, CRANFIELD UNIVERSITY        #
-#  Created on behalf of the IFRA Group at Cranfield University, United Kingdom          #
-#  E-mail: IFRA@cranfield.ac.uk                                                         #
-#                                                                                       #
-#  Licensed under the Apache-2.0 License.                                               #
-#  You may not use this file except in compliance with the License.                     #
-#  You may obtain a copy of the License at: http://www.apache.org/licenses/LICENSE-2.0  #
-#                                                                                       #
-#  Unless required by applicable law or agreed to in writing, software distributed      #
-#  under the License is distributed on an "as-is" basis, without warranties or          #
-#  conditions of any kind, either express or implied. See the License for the specific  #
-#  language governing permissions and limitations under the License.                    #
-#                                                                                       #
-#  IFRA Group - Cranfield University                                                    #
-#  AUTHORS: Mikel Bueno Viso - Mikel.Bueno-Viso@cranfield.ac.uk                         #
-#           Seemal Asif      - s.asif@cranfield.ac.uk                                   #
-#           Phil Webb        - p.f.webb@cranfield.ac.uk                                 #
-#                                                                                       #
-#  Date: July, 2022.                                                                    #
-#                                                                                       #
-# ===================================== COPYRIGHT ===================================== #
-# ===================================== COPYRIGHT ===================================== #
-#                                                                                       #
-#  Some of the information used to build the ROS2 ABB-IRB120 .urdf files in this ROS2   #
-#  repository has been taken from the following resource:                               #
-#       - abb_experimental (https://github.com/ros-industrial/abb_experimental)         #
-#                                                                                       #
-#  AUTHORS:                                                                             #
-#       - ROS-Industrial - https://rosindustrial.org                                    #
-#       - Mark Culleton (Trinity College Dublin) - culletom@tcd.ie                      #
-#       - Kevin Kelly   (Trinity College Dublin)                                        #
-#                                                                                       #
-#  COPYRIGHT - ROS-Industrial                                                           #
-#  (ORIGINAL LICENSE) -> Licensed under the Apache-2.0 License.                         #
-#                                                                                       #
-#  CHANGES MADE:                                                                        #
-#  The original files contain the .urdf information of the robot for ROS1, and these    #
-#  have been modified for ROS2.                                                         #
-#                                                                                       #
-# ===================================== COPYRIGHT ===================================== #
-# ======= CITE OUR WORK ======= #
-# You can cite our work with the following statement:
-# IFRA (2022) ROS2.0 ROBOT SIMULATION. URL: https://github.com/IFRA-Cranfield/ros2_RobotSimulation.
--->
 <robot name="irb120" xmlns:xacro="http://ros.org/wiki/xacro">
-  <!-- ===== ARGUMENTS ===== -->
-  <!-- CELL LAYOUT:  -->
   <xacro:arg name="cell_layout_1" default="false"/>
   <xacro:property name="cell_layout_1" value="$(arg cell_layout_1)"/>
@@ -56,10 +7,8 @@
   <xacro:arg name="cell_layout_3" default="false"/>
   <xacro:property name="cell_layout_3" value="$(arg cell_layout_3)"/>
-  <!-- END-EFFECTOR:  -->
   <xacro:arg name="EE_no" default="false"/>
   <xacro:property name="EE_no" value="$(arg EE_no)"/>
   <xacro:arg name="EE_schunk" default="false"/>
   <xacro:property name="EE_schunk" value="$(arg EE_schunk)"/>
-  <!-- Include XACRO-MACRO file of the IRB120: -->
   <xacro:include filename="$(find irb120_ros2_gazebo)/urdf/irb120_macro.urdf.xacro"/>
   <xacro:irb120
@@ -68,9 +17,5 @@
     EE_schunk="${EE_schunk}"
   />
-  <!-- Gazebo WORLD link: -->
   <link name="world"/>
-  <!-- ========== ========== ========== ========== ========== ========== -->
-  <!-- CELL LAYOUT SELECTION: -->
-  <!-- CELL LAYOUT N1) ABB IRB120 Robot alone: -->
   <xacro:if value="${cell_layout_1}">
     <joint name="world-base_link-fixed" type="fixed">
@@ -79,5 +24,4 @@
     </joint>
   </xacro:if>
-  <!-- CELL LAYOUT N2) ABB IRB120 Robot in Cranfield University cell: -->
   <xacro:if value="${cell_layout_2}">
     <link name="cell">
@@ -109,5 +53,4 @@
     </joint>
   </xacro:if>
-  <!-- CELL LAYOUT N3) ABB IRB120 + PICK & PLACE layout: -->
   <xacro:if value="${cell_layout_3}">
     <link name='irb120_block'>

File: ABBRobots/IRB120/irb120_ros2_gazebo/urdf/irb120_macro.urdf.xacro (robot description, xacro)
@@ -1,56 +1,6 @@
 <?xml version="1.0"?>
-<!--
-# ===================================== COPYRIGHT ===================================== #
-#                                                                                       #
-#  IFRA (Intelligent Flexible Robotics and Assembly) Group, CRANFIELD UNIVERSITY        #
-#  Created on behalf of the IFRA Group at Cranfield University, United Kingdom          #
-#  E-mail: IFRA@cranfield.ac.uk                                                         #
-#                                                                                       #
-#  Licensed under the Apache-2.0 License.                                               #
-#  You may not use this file except in compliance with the License.                     #
-#  You may obtain a copy of the License at: http://www.apache.org/licenses/LICENSE-2.0  #
-#                                                                                       #
-#  Unless required by applicable law or agreed to in writing, software distributed      #
-#  under the License is distributed on an "as-is" basis, without warranties or          #
-#  conditions of any kind, either express or implied. See the License for the specific  #
-#  language governing permissions and limitations under the License.                    #
-#                                                                                       #
-#  IFRA Group - Cranfield University                                                    #
-#  AUTHORS: Mikel Bueno Viso - Mikel.Bueno-Viso@cranfield.ac.uk                         #
-#           Seemal Asif      - s.asif@cranfield.ac.uk                                   #
-#           Phil Webb        - p.f.webb@cranfield.ac.uk                                 #
-#                                                                                       #
-#  Date: July, 2022.                                                                    #
-#                                                                                       #
-# ===================================== COPYRIGHT ===================================== #
-# ===================================== COPYRIGHT ===================================== #
-#                                                                                       #
-#  Some of the information used to build the ROS2 ABB-IRB120 .urdf files in this ROS2   #
-#  repository has been taken from the following resource:                               #
-#       - abb_experimental (https://github.com/ros-industrial/abb_experimental)         #
-#                                                                                       #
-#  AUTHORS:                                                                             #
-#       - ROS-Industrial - https://rosindustrial.org                                    #
-#       - Mark Culleton (Trinity College Dublin) - culletom@tcd.ie                      #
-#       - Kevin Kelly   (Trinity College Dublin)                                        #
-#                                                                                       #
-#  COPYRIGHT - ROS-Industrial                                                           #
-#  (ORIGINAL LICENSE) -> Licensed under the Apache-2.0 License.                         #
-#                                                                                       #
-#  CHANGES MADE:                                                                        #
-#  The original files contain the .urdf information of the robot for ROS1, and these    #
-#  have been modified for ROS2.                                                         #
-#                                                                                       #
-# ===================================== COPYRIGHT ===================================== #
-# ======= CITE OUR WORK ======= #
-# You can cite our work with the following statement:
-# IFRA (2022) ROS2.0 ROBOT SIMULATION. URL: https://github.com/IFRA-Cranfield/ros2_RobotSimulation.
--->
 <robot xmlns:xacro="http://ros.org/wiki/xacro">
-  <!-- Include additional ABB-Resources/MATERIALS+COLOUR xacro files: -->
   <xacro:include filename="$(find irb120_ros2_gazebo)/urdf/abb_resources/common_materials.xacro"/>
-  <!-- XACRO-MACRO of ABB-IRB120: -->
   <xacro:macro name="irb120" params="prefix EE_no EE_schunk">
-    <!-- Load ABB IRB120 TRANSMISSION file: -->
     <xacro:include filename="$(find irb120_ros2_gazebo)/urdf/irb120_transmission.xacro" />
     <xacro:irb120_transmission
@@ -58,5 +8,4 @@
       EE_schunk="${EE_schunk}"
     />
-    <!-- Load ABB IRB120 ROS2_CONTROL file: -->
     <xacro:include filename="$(find irb120_ros2_gazebo)/urdf/irb120_ros2control.xacro" />
     <xacro:irb120_ros2control
@@ -65,8 +14,5 @@
       EE_schunk="${EE_schunk}"
     />
-    <!-- ***** ABB-IRB120 ROBOT .urdf SERIAL CHAIN ***** -->
-    <!-- Link list: -->
-    <!-- base_link -->
-    <link name="${prefix}base_link">
+    <link name="base_link">
       <inertial>
         <mass value="6.215"/>
@@ -89,6 +35,5 @@
       </collision>
     </link>
-    <!-- link_1 -->
-    <link name="${prefix}link_1">
+    <link name="link_1">
       <inertial>
         <mass value="3.067" />
@@ -111,6 +56,5 @@
       </collision>
     </link>
-    <!-- link_2 -->
-    <link name="${prefix}link_2">
+    <link name="link_2">
       <inertial>
         <mass value="3.909"/>
@@ -133,6 +77,5 @@
       </collision>
     </link>
-    <!-- link_3 -->
-    <link name="${prefix}link_3">
+    <link name="link_3">
       <inertial>
         <mass value="2.944"/>
@@ -155,6 +98,5 @@
       </collision>
     </link>
-    <!-- link_4 -->
-    <link name="${prefix}link_4">
+    <link name="link_4">
       <inertial>
         <mass value="1.328"/>
@@ -177,6 +119,5 @@
       </collision>
     </link>
-    <!-- link_5 -->
-    <link name="${prefix}link_5">
+    <link name="link_5">
       <inertial>
         <mass value="0.546"/>
@@ -199,6 +140,5 @@
       </collision>
     </link>
-    <!-- link_6 -->
-    <link name="${prefix}link_6">
+    <link name="link_6">
       <inertial>
         <mass value="0.137"/>
@@ -221,87 +161,71 @@
       </collision>
     </link>
-    <!-- end of link list -->
-    <!-- Joint list: -->
-    <!-- joint_1 -->
-    <joint name="${prefix}joint_1" type="revolute">
+    <joint name="joint_1" type="revolute">
       <origin rpy="0 0 0" xyz="0 0 0"/>
-      <parent link="${prefix}base_link"/>
-      <child link="${prefix}link_1"/>
+      <parent link="base_link"/>
+      <child link="link_1"/>
       <limit effort="0" lower="-2.87979" upper="2.87979" velocity="4.36332"/>
       <axis xyz="0 0 1"/>
       <dynamics damping="0.0" friction="0.0"/>
     </joint>
-    <!-- joint_2 -->
-    <joint name="${prefix}joint_2" type="revolute">
+    <joint name="joint_2" type="revolute">
       <origin rpy="0 0 0" xyz="0 0 0.29"/>
-      <parent link="${prefix}link_1"/>
-      <child link="${prefix}link_2"/>
+      <parent link="link_1"/>
+      <child link="link_2"/>
       <limit effort="0" lower="-1.91986" upper="1.91986" velocity="4.36332"/>
       <axis xyz="0 1 0"/>
       <dynamics damping="0.0" friction="0.0"/>
     </joint>
-    <!-- joint_3 -->
-    <joint name="${prefix}joint_3" type="revolute">
+    <joint name="joint_3" type="revolute">
       <origin rpy="0 0 0" xyz="0 0 0.27"/>
-      <parent link="${prefix}link_2"/>
-      <child link="${prefix}link_3"/>
+      <parent link="link_2"/>
+      <child link="link_3"/>
       <limit effort="0" lower="-1.91986" upper="1.22173" velocity="4.36332"/>
       <axis xyz="0 1 0"/>
       <dynamics damping="0.0" friction="0.0"/>
     </joint>
-    <!-- joint_4 -->
-    <joint name="${prefix}joint_4" type="revolute">
+    <joint name="joint_4" type="revolute">
       <origin rpy="0 0 0" xyz="0 0 0.07"/>
-      <parent link="${prefix}link_3"/>
-      <child link="${prefix}link_4"/>
+      <parent link="link_3"/>
+      <child link="link_4"/>
       <limit effort="0" lower="-2.79253" upper="2.79253" velocity="5.58505"/>
       <axis xyz="1 0 0"/>
       <dynamics damping="0.0" friction="0.0"/>
     </joint>
-    <!-- joint_5 -->
-    <joint name="${prefix}joint_5" type="revolute">
+    <joint name="joint_5" type="revolute">
       <origin rpy="0 0 0" xyz="0.302 0 0"/>
-      <parent link="${prefix}link_4"/>
-      <child link="${prefix}link_5"/>
+      <parent link="link_4"/>
+      <child link="link_5"/>
       <limit effort="0" lower="-2.094395" upper="2.094395" velocity="5.58505"/>
       <axis xyz="0 1 0"/>
       <dynamics damping="0.0" friction="0.0"/>
     </joint>
-    <!-- joint_6 -->
-    <joint name="${prefix}joint_6" type="revolute">
+    <joint name="joint_6" type="revolute">
       <origin rpy="0 0 0" xyz="0.072 0 0"/>
-      <parent link="${prefix}link_5"/>
-      <child link="${prefix}link_6"/>
+      <parent link="link_5"/>
+      <child link="link_6"/>
       <limit effort="0" lower="-6.98132" upper="6.98132" velocity="7.33038"/>
       <axis xyz="1 0 0"/>
       <dynamics damping="0.0" friction="0.0"/>
     </joint>
-    <!-- end of joint list -->
-    <!-- ROS-Industrial 'base' frame: base_link to ABB World Coordinates transform -->
-    <link name="${prefix}base" />
-    <joint name="${prefix}base_link-base" type="fixed">
+    <link name="base" />
+    <joint name="base_link-base" type="fixed">
       <origin xyz="0 0 0" rpy="0 0 0"/>
-      <parent link="${prefix}base_link"/>
-      <child link="${prefix}base"/>
-    </joint>
-    <!-- ROS-Industrial 'flange' frame: attachment point for EEF models -->
-    <link name="${prefix}flange"/>
-    <joint type="fixed" name="${prefix}joint_6-flange">
+      <parent link="base_link"/>
+      <child link="base"/>
+    </joint>
+    <link name="flange"/>
+    <joint type="fixed" name="joint_6-flange">
       <origin xyz="0 0 0" rpy="0 0 0"/>
-      <parent link="${prefix}link_6"/>
-      <child link="${prefix}flange"/>
-    </joint>
-    <!-- ROS-Industrial 'tool0' frame: all-zeros tool frame -->
-    <link name="${prefix}tool0" />
-    <joint name="${prefix}link_6-tool0" type="fixed">
+      <parent link="link_6"/>
+      <child link="flange"/>
+    </joint>
+    <link name="tool0" />
+    <joint name="link_6-tool0" type="fixed">
       <origin xyz="0 0 0" rpy="0 ${radians(90)} 0" />
-      <parent link="${prefix}flange" />
-      <child link="${prefix}tool0" />
-    </joint>
-    <!-- =================================== -->
-    <!-- ========== END-EFFECTORS ========== -->
-    <!-- === SCHUNK EGP-64 GRIPPER === -->
+      <parent link="flange" />
+      <child link="tool0" />
+    </joint>
     <xacro:if value="${EE_schunk}">
-      <!-- Schunk coupler (LINK): -->
       <link name="schunk_coupler">
         <visual>
@@ -321,5 +245,4 @@
         </inertial>
       </link>
-      <!-- Schunk coupler (JOINT): -->
       <joint name="schunk_coupler_joint" type="fixed">
         <origin xyz="0 0 0.001" rpy="0 0 ${pi/4}" />
@@ -358,5 +281,4 @@
         <origin xyz="-0.03205 0.01812 0.02047" rpy="0 0 0" />
       </joint>
-      <!-- LEFT FINGER BASE -->
       <link name="egp64_finger_left_link">
         <inertial>
@@ -387,5 +309,4 @@
         <axis xyz="-1 0 0" />
       </joint>
-      <!-- LEFT FINGERTIP -->
       <link name="egp64_fingertip_left_link">
         <inertial>
@@ -414,5 +335,4 @@
         <origin xyz="0.03869 -0.0005 0.00093" rpy="0 0 0"/>
       </joint>
-      <!-- RIGHT FINGER BASE -->
       <link name="egp64_finger_right_link">
         <inertial>
@@ -441,5 +361,4 @@
         <axis xyz="1 0 0" />
       </joint>
-      <!-- RIGHT FINGERTIP -->
       <link name="egp64_fingertip_right_link">
         <inertial>
@@ -466,5 +385,4 @@
         <origin xyz="-0.01211 -0.00197 0.00093" rpy="0 0 0"/>
       </joint>
-      <!-- SMALL CUBE FOR GRIPPER PLUGIN -->
       <link name="EE_egp64">
         <inertial>
@@ -487,5 +405,4 @@
       </joint>
     </xacro:if>
-    <!-- === SCHUNK EGP-64 GRIPPER === -->
   </xacro:macro>
 </robot>
