Commit message: add all changes

File: ABBRobots/IRB120/irb120_ros2_gazebo/urdf/irb120_ros2control.xacro (robot description, xacro)
@@ -1,80 +1,25 @@
 <?xml version="1.0"?>
-<!--
-# ===================================== COPYRIGHT ===================================== #
-#                                                                                       #
-#  IFRA (Intelligent Flexible Robotics and Assembly) Group, CRANFIELD UNIVERSITY        #
-#  Created on behalf of the IFRA Group at Cranfield University, United Kingdom          #
-#  E-mail: IFRA@cranfield.ac.uk                                                         #
-#                                                                                       #
-#  Licensed under the Apache-2.0 License.                                               #
-#  You may not use this file except in compliance with the License.                     #
-#  You may obtain a copy of the License at: http://www.apache.org/licenses/LICENSE-2.0  #
-#                                                                                       #
-#  Unless required by applicable law or agreed to in writing, software distributed      #
-#  under the License is distributed on an "as-is" basis, without warranties or          #
-#  conditions of any kind, either express or implied. See the License for the specific  #
-#  language governing permissions and limitations under the License.                    #
-#                                                                                       #
-#  IFRA Group - Cranfield University                                                    #
-#  AUTHORS: Mikel Bueno Viso - Mikel.Bueno-Viso@cranfield.ac.uk                         #
-#           Seemal Asif      - s.asif@cranfield.ac.uk                                   #
-#           Phil Webb        - p.f.webb@cranfield.ac.uk                                 #
-#                                                                                       #
-#  Date: July, 2022.                                                                    #
-#                                                                                       #
-# ===================================== COPYRIGHT ===================================== #
-# ===================================== COPYRIGHT ===================================== #
-#                                                                                       #
-#  Some of the information used to build the ROS2 ABB-IRB120 .urdf files in this ROS2   #
-#  repository has been taken from the following resource:                               #
-#       - abb_experimental (https://github.com/ros-industrial/abb_experimental)         #
-#                                                                                       #
-#  AUTHORS:                                                                             #
-#       - ROS-Industrial - https://rosindustrial.org                                    #
-#       - Mark Culleton (Trinity College Dublin) - culletom@tcd.ie                      #
-#       - Kevin Kelly   (Trinity College Dublin)                                        #
-#                                                                                       #
-#  COPYRIGHT - ROS-Industrial                                                           #
-#  (ORIGINAL LICENSE) -> Licensed under the Apache-2.0 License.                         #
-#                                                                                       #
-#  CHANGES MADE:                                                                        #
-#  The original files contain the .urdf information of the robot for ROS1, and these    #
-#  have been modified for ROS2.                                                         #
-#                                                                                       #
-# ===================================== COPYRIGHT ===================================== #
-# ======= CITE OUR WORK ======= #
-# You can cite our work with the following statement:
-# IFRA (2022) ROS2.0 ROBOT SIMULATION. URL: https://github.com/IFRA-Cranfield/ros2_RobotSimulation.
--->
 <robot xmlns:xacro="http://www.ros.org/wiki/xacro">
   <xacro:macro name="irb120_ros2control" params="prefix EE_no EE_schunk" >
-    <!-- ROS2_CONTROL tag name: -->
-    <xacro:property name="name" value="GazeboSystem"/>
-    <!-- ===== Gazebo ROS2_CONTROL plugin ===== -->
-    <!-- No End-Effector: -->
+    <xacro:property name="name" value="GazeboSimSystem"/>
     <xacro:if value="${EE_no}">
       <gazebo>
-        <plugin filename="libgazebo_ros2_control.so" name="gazebo_ros2_control">
-          <robot_sim_type>gazebo_ros2_control/GazeboSystem</robot_sim_type>
-          <parameters>$(find irb120_ros2_gazebo)/config/irb120_controller.yaml</parameters>
+        <plugin filename="libgz_ros22_control.so" name="gz_ros22_control">
+          <parameters>/home/dina2997/master_ws/src/ros2_RobotSimulation/ABBRobots/IRB120/irb120_ros2_gazebo/config/irb120_controller.yaml</parameters>
         </plugin>
       </gazebo>
     </xacro:if>
-    <!-- End-Effector -> SCHUNK EGP-64 GRIPPER: -->
     <xacro:if value="${EE_schunk}">
       <gazebo>
-        <plugin filename="libgazebo_ros2_control.so" name="gazebo_ros2_control">
-          <robot_sim_type>gazebo_ros2_control/GazeboSystem</robot_sim_type>
-          <parameters>$(find irb120_ros2_gazebo)/config/irb120egp64_controller.yaml</parameters>
+        <plugin filename="libgz_ros22_control.so" name="gz_ros22_control">
+          <parameters>/home/dina2997/master_ws/src/ros2_RobotSimulation/ABBRobots/IRB120/irb120_ros2_gazebo/config/irb120egp64_controller.yaml</parameters>
         </plugin>
       </gazebo>
     </xacro:if>
-    <!-- ========== ROS2 CONTROL ========== -->
     <ros2_control name="${name}" type="system">
       <hardware>
-        <plugin>gazebo_ros2_control/GazeboSystem</plugin>
+        <plugin>gz_ros2_control/GazeboSimSystem</plugin>
       </hardware>
-      <!-- irb120_joint1 -->
-      <joint name="${prefix}joint_1">
+      <joint name="joint_1">
         <command_interface name="position">
           <param name="min">-2.87979</param>
@@ -89,6 +34,5 @@
         <state_interface name="effort"/>
       </joint>
-      <!-- irb120_joint2 -->
-      <joint name="${prefix}joint_2">
+      <joint name="joint_2">
         <command_interface name="position">
           <param name="min">-1.91986</param>
@@ -103,6 +47,5 @@
         <state_interface name="effort"/>
       </joint>
-      <!-- irb120_joint3 -->
-      <joint name="${prefix}joint_3">
+      <joint name="joint_3">
         <command_interface name="position">
           <param name="min">-1.91986</param>
@@ -117,6 +60,5 @@
         <state_interface name="effort"/>
       </joint>
-      <!-- irb120_joint4 -->
-      <joint name="${prefix}joint_4">
+      <joint name="joint_4">
         <command_interface name="position">
           <param name="min">-2.79253</param>
@@ -131,6 +73,5 @@
         <state_interface name="effort"/>
       </joint>
-      <!-- irb120_joint5 -->
-      <joint name="${prefix}joint_5">
+      <joint name="joint_5">
         <command_interface name="position">
           <param name="min">-2.094395</param>
@@ -145,6 +86,5 @@
         <state_interface name="effort"/>
       </joint>
-      <!-- irb120_joint6 -->
-      <joint name="${prefix}joint_6">
+      <joint name="joint_6">
         <command_interface name="position">
           <param name="min">-6.98132</param>
@@ -159,9 +99,5 @@
         <state_interface name="effort"/>
       </joint>
-      <!-- =================================== -->
-      <!-- ========== END-EFFECTORS ========== -->
-      <!-- === SCHUNK EGP-64 GRIPPER === -->
       <xacro:if value="${EE_schunk}">
-        <!-- egp64_finger_left_joint -->
         <joint name="egp64_finger_left_joint">
           <command_interface name="position">
@@ -176,5 +112,4 @@
           <state_interface name="velocity"/>
         </joint>
-        <!-- egp64_finger_right_joint -->
         <joint name="egp64_finger_right_joint">
           <command_interface name="position">
@@ -204,37 +139,33 @@
         </joint>
       </xacro:if>
-      <!-- === SCHUNK EGP-64 GRIPPER === -->
     </ros2_control>
-    <gazebo reference="${prefix}base_link">
+    <gazebo reference="base_link">
       <selfCollide>false</selfCollide>
       <material>Gazebo/Orange</material>
     </gazebo>
-    <gazebo reference="${prefix}link_1">
+    <gazebo reference="link_1">
       <selfCollide>false</selfCollide>
       <material>Gazebo/Orange</material>
     </gazebo>
-    <gazebo reference="${prefix}link_2">
+    <gazebo reference="link_2">
       <selfCollide>false</selfCollide>
       <material>Gazebo/Orange</material>
     </gazebo>
-    <gazebo reference="${prefix}link_3">
+    <gazebo reference="link_3">
       <selfCollide>false</selfCollide>
       <material>Gazebo/Orange</material>
     </gazebo>
-    <gazebo reference="${prefix}link_4">
+    <gazebo reference="link_4">
       <selfCollide>false</selfCollide>
       <material>Gazebo/Orange</material>
     </gazebo>
-    <gazebo reference="${prefix}link_5">
+    <gazebo reference="link_5">
       <selfCollide>false</selfCollide>
       <material>Gazebo/Orange</material>
     </gazebo>
-    <gazebo reference="${prefix}link_6">
+    <gazebo reference="link_6">
       <selfCollide>false</selfCollide>
       <material>Gazebo/Orange</material>
     </gazebo>
-    <!-- =================================== -->
-    <!-- ========== END-EFFECTORS ========== -->
-    <!-- === SCHUNK EGP-64 GRIPPER === -->
     <xacro:if value="${EE_schunk}">
       <gazebo reference="egp64_gripper_base_link">
@@ -254,8 +185,6 @@
       </gazebo>
     </xacro:if>
-    <!-- === SCHUNK EGP-64 GRIPPER === -->
     <gazebo reference="end_effector_frame_fixed_joint">
       <preserveFixedJoint>true</preserveFixedJoint>
-      <!-- For compatibility with SDFormat < 4.4 -->
       <disableFixedJointLumping>true</disableFixedJointLumping>
     </gazebo>

File: ABBRobots/IRB120/irb120_ros2_gazebo/urdf/irb120_transmission.xacro (robot description, xacro)
@@ -1,115 +1,65 @@
 <?xml version="1.0"?>
-<!--
-# ===================================== COPYRIGHT ===================================== #
-#                                                                                       #
-#  IFRA (Intelligent Flexible Robotics and Assembly) Group, CRANFIELD UNIVERSITY        #
-#  Created on behalf of the IFRA Group at Cranfield University, United Kingdom          #
-#  E-mail: IFRA@cranfield.ac.uk                                                         #
-#                                                                                       #
-#  Licensed under the Apache-2.0 License.                                               #
-#  You may not use this file except in compliance with the License.                     #
-#  You may obtain a copy of the License at: http://www.apache.org/licenses/LICENSE-2.0  #
-#                                                                                       #
-#  Unless required by applicable law or agreed to in writing, software distributed      #
-#  under the License is distributed on an "as-is" basis, without warranties or          #
-#  conditions of any kind, either express or implied. See the License for the specific  #
-#  language governing permissions and limitations under the License.                    #
-#                                                                                       #
-#  IFRA Group - Cranfield University                                                    #
-#  AUTHORS: Mikel Bueno Viso - Mikel.Bueno-Viso@cranfield.ac.uk                         #
-#           Seemal Asif      - s.asif@cranfield.ac.uk                                   #
-#           Phil Webb        - p.f.webb@cranfield.ac.uk                                 #
-#                                                                                       #
-#  Date: July, 2022.                                                                    #
-#                                                                                       #
-# ===================================== COPYRIGHT ===================================== #
-# ===================================== COPYRIGHT ===================================== #
-#                                                                                       #
-#  Some of the information used to build the ROS2 ABB-IRB120 .urdf files in this ROS2   #
-#  repository has been taken from the following resource:                               #
-#       - abb_experimental (https://github.com/ros-industrial/abb_experimental)         #
-#                                                                                       #
-#  AUTHORS:                                                                             #
-#       - ROS-Industrial - https://rosindustrial.org                                    #
-#       - Mark Culleton (Trinity College Dublin) - culletom@tcd.ie                      #
-#       - Kevin Kelly   (Trinity College Dublin)                                        #
-#                                                                                       #
-#  COPYRIGHT - ROS-Industrial                                                           #
-#  (ORIGINAL LICENSE) -> Licensed under the Apache-2.0 License.                         #
-#                                                                                       #
-#  CHANGES MADE:                                                                        #
-#  The original files contain the .urdf information of the robot for ROS1, and these    #
-#  have been modified for ROS2.                                                         #
-#                                                                                       #
-# ===================================== COPYRIGHT ===================================== #
-# ======= CITE OUR WORK ======= #
-# You can cite our work with the following statement:
-# IFRA (2022) ROS2.0 ROBOT SIMULATION. URL: https://github.com/IFRA-Cranfield/ros2_RobotSimulation.
--->
 <robot xmlns:xacro="http://wiki.ros.org/xacro">
   <xacro:macro name="irb120_transmission" params="prefix EE_schunk">
-    <transmission name="irb120_joint1_trans">
+    <transmission name="joint_1_trans">
       <type>transmission_interface/SimpleTransmission</type>
-      <joint name="${prefix}irb120_joint1">
+      <joint_ name="joint_1">
         <hardwareInterface>hardware_interface/PositionJointInterface</hardwareInterface>
-      </joint>
-      <actuator name="irb120_joint1_motor">
+      </joint_>
+      <actuator name="joint_1_motor">
         <mechanicalReduction>1</mechanicalReduction>
       </actuator>
     </transmission>
-    <transmission name="irb120_joint2_trans">
+    <transmission name="joint_2_trans">
       <type>transmission_interface/SimpleTransmission</type>
-      <joint name="${prefix}irb120_joint2">
+      <joint_ name="joint_2">
         <hardwareInterface>hardware_interface/PositionJointInterface</hardwareInterface>
-      </joint>
-      <actuator name="irb120_joint2_motor">
+      </joint_>
+      <actuator name="joint_2_motor">
         <mechanicalReduction>1</mechanicalReduction>
       </actuator>
     </transmission>
-    <transmission name="irb120_joint3_trans">
+    <transmission name="joint_3_trans">
       <type>transmission_interface/SimpleTransmission</type>
-      <joint name="${prefix}irb120_joint3">
+      <joint_ name="joint_3">
         <hardwareInterface>hardware_interface/PositionJointInterface</hardwareInterface>
-      </joint>
-      <actuator name="irb120_joint3_motor">
+      </joint_>
+      <actuator name="joint_3_motor">
         <mechanicalReduction>1</mechanicalReduction>
       </actuator>
     </transmission>
-    <transmission name="irb120_joint4_trans">
+    <transmission name="joint_4_trans">
       <type>transmission_interface/SimpleTransmission</type>
-      <joint name="${prefix}irb120_joint4">
+      <joint_ name="joint_4">
         <hardwareInterface>hardware_interface/PositionJointInterface</hardwareInterface>
-      </joint>
-      <actuator name="irb120_joint4_motor">
+      </joint_>
+      <actuator name="joint_4_motor">
         <mechanicalReduction>1</mechanicalReduction>
       </actuator>
     </transmission>
-    <transmission name="irb120_joint5_trans">
+    <transmission name="joint_5_trans">
       <type>transmission_interface/SimpleTransmission</type>
-      <joint name="${prefix}irb120_joint5">
+      <joint_ name="joint_5">
         <hardwareInterface>hardware_interface/PositionJointInterface</hardwareInterface>
-      </joint>
-      <actuator name="irb120_joint5_motor">
+      </joint_>
+      <actuator name="joint_5_motor">
         <mechanicalReduction>1</mechanicalReduction>
       </actuator>
     </transmission>
-    <transmission name="irb120_joint6_trans">
+    <transmission name="joint_6_trans">
       <type>transmission_interface/SimpleTransmission</type>
-      <joint name="${prefix}irb120_joint6">
+      <joint_ name="joint_6">
         <hardwareInterface>hardware_interface/PositionJointInterface</hardwareInterface>
-      </joint>
-      <actuator name="irb120_joint6_motor">
+      </joint_>
+      <actuator name="joint_6_motor">
         <mechanicalReduction>1</mechanicalReduction>
       </actuator>
     </transmission>
-    <!-- =================================== -->
-    <!-- ========== END-EFFECTORS ========== -->
-    <!-- === SCHUNK EGP-64 GRIPPER === -->
     <xacro:if value="${EE_schunk}">
       <transmission name="egp64_left_finger_trans">
         <type>transmission_interface/SimpleTransmission</type>
-        <joint name="egp64_finger_left_joint">
+        <joint_ name="egp64_finger_left_joint_">
           <hardwareInterface>hardware_interface/PositionJointInterface</hardwareInterface>
-        </joint>
+        </joint_>
         <actuator name="egp64_left_finger_motor">
           <mechanicalReduction>1</mechanicalReduction>
@@ -118,7 +68,7 @@
       <transmission name="egp64_right_finger_trans">
         <type>transmission_interface/SimpleTransmission</type>
-        <joint name="egp64_finger_right_joint">
+        <joint_ name="egp64_finger_right_joint_">
           <hardwareInterface>hardware_interface/PositionJointInterface</hardwareInterface>
-        </joint>
+        </joint_>
         <actuator name="egp64_right_finger_motor">
           <mechanicalReduction>1</mechanicalReduction>
@@ -126,5 +76,4 @@
       </transmission>
     </xacro:if>
-    <!-- === SCHUNK EGP-64 GRIPPER === -->
   </xacro:macro>
 </robot>
